File: hardware/multi-touch-v2.kicad_pcb (KiCad board)
At the start: 2 copper layers, 25 x 30 mm, 27 parts, among them P1 CON-SENSOR2, P2 DEBUG, P3 BOOT, P4 CONN_01X12, U1 CPT112S, U2 XMC1XXX24, U3 DRILL, U4 DRILL, U5 DRILL, U6 DRILL

Commit message: Add layout
Parts:
- removed R3, R4: TBD, kicad-libraries:R0603F
- added D1: blue, kicad-libraries:D0603F, F.Cu at (58.7, 31.6)
- added G***: LOGO, kicad-libraries:Logo_CoMCU, B.Cu at (46.5, 35.9)
- added RP2: TBD (2k2), kicad-libraries:4X0402, F.Cu at (55.0, 47.2)
- P4: footprint pin_array_6x2 -> kicad-libraries:pin_array_6x2
- R1: value 75k -> 1k; footprint kicad-libraries:R0603 -> kicad-libraries:R0603F
- U1: footprint kicad-libraries:SOIC8 -> kicad-libraries:QFN-20-3x3
- moved R5 37.4 mm to (52.1, 30.2)
- moved D2 36.0 mm to (52.1, 31.6)
- moved C4 32.0 mm to (50.0, 35.9), turned to 270 degrees
- moved C6 27.1 mm to (49.6, 41.0), turned to 270 degrees
- moved P4 26.0 mm to (61.9, 42.3), turned to 90 degrees
- moved P3 19.4 mm to (45.9, 50.6)
- moved Fiducial_Mark 19.1 mm to (62.9, 33.3)
- moved R1 17.2 mm to (58.7, 30.2), turned to 0 degrees
- moved P2 16.1 mm to (59.3, 51.9)
- moved C5 13.3 mm to (50.7, 55.0), turned to 180 degrees
- moved Fiducial_Mark 10.6 mm to (44.9, 45.3)
- moved VAL 10.4 mm to (46.4, 42.6), turned to 180 degrees
- moved U2 10.1 mm to (50.7, 51.7), turned to 0 degrees
- moved VAL 9.40 mm to (46.5, 49.6), turned to 180 degrees
- moved C1 8.52 mm to (50.9, 41.0)
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Connections:
- R1 pad 2: GND -> Net-(D1-Pad2)
- U1 pad 1: Net-(P4-Pad2) -> Net-(P4-Pad11)
- U1 pad 2: Net-(P4-Pad1) -> Net-(P4-Pad12)
- U1 pad 5: Net-(U1-Pad5) -> SCL_Conf
- U1 pad 6: Net-(U1-Pad6) -> SDA-Conf
- U2 pad 12: Net-(U2-Pad12) -> SCL_Conf
- U2 pad 14: Net-(U2-Pad14) -> Net-(R1-Pad1)
- U2 pad 16: Net-(U2-Pad16) -> Net-(R5-Pad1)
- U2 pad 18: INT -> SDA-Conf
- U2 pad 20: Net-(U2-Pad20) -> INT
- U2 pad 7: Net-(R5-Pad1) -> Net-(U2-Pad7)
Routing:
- net (no net): track 53.6 -> 0.00 mm
- net GND: track 78.0 -> 33.1 mm, vias 8 -> 11
- net VCC: track 108.6 -> 65.8 mm, vias 17 -> 3
- net Net-(R5-Pad1): track 0.00 -> 28.9 mm, vias 0 -> 2
- net Net-(R1-Pad1): track 3.39 -> 30.6 mm, vias 0 -> 2
- net SCL_Conf: track 0.00 -> 18.0 mm, vias 0 -> 3
- net Net-(P1-Pad5): track 20.7 -> 5.00 mm, vias 3 -> 0
- net Net-(U1-Pad5): track 14.8 -> 0.00 mm, vias 2 -> 0
- net SDA-Conf: track 0.00 -> 14.3 mm, vias 0 -> 4
- net S-MOSI: track 15.8 -> 1.60 mm, vias 2 -> 0
- net Net-(P4-Pad11): track 0.00 -> 13.2 mm
- net Net-(C2-Pad1): track 15.5 -> 2.23 mm, vias 3 -> 0
- net SCL: track 0.00 -> 12.8 mm, vias 0 -> 2
- net Net-(P4-Pad3): track 0.00 -> 12.5 mm
- net Net-(P4-Pad9): track 0.00 -> 12.4 mm
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- removed copper zone on F.Cu, net GND
Other:
- rule via_min_size: 0.70104 -> 0.5
- board text added: "Multi Touch 2.0"
- board text added: "Status"
- board text added: "Touch"
- board text removed: "Multi Touch 1.0"

Commit message: Fix page settings
Other:
- board text added: "Copyright Tinkerforge GmbH 2018. This documentation describes Open Hardware and is licensed under the CERN OHL v. 1.1. You may redistribute and modify this documentation under the terms of the CERN OHL v.1.1. (http://ohwr.org/cernohl). This documentation is distributed WITHOUT ANY EXPRESS OR IMPLIED WARRANTY, INCLUDING OF MERCHANTABILITY, SATISFACTORY QUALITY AND FITNESS FOR A PARTICULAR PURPOSE.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"
- board text removed: "Copyright Tinkerforge GmbH 2013. This documentation describes Open Hardware and is licensed under the CERN OHL v. 1.1. You may redistribute and modify this documentation under the terms of the CERN OHL v.1.1. (http://ohwr.org/cernohl). This documentation is distributed WITHOUT ANY EXPRESS OR IMPLIED WARRANTY, INCLUDING OF MERCHANTABILITY, SATISFACTORY QUALITY AND FITNESS FOR A PARTICULAR PURPOSE.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"
Changed lines of the file:
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@@
-(kicad_pcb (version 4) (host pcbnew 4.0.2+dfsg1-stable)
+(kicad_pcb (version 4) (host pcbnew 4.0.7+dfsg1-1ubuntu2)
   (general
     (links 69)
     (no_connects 0)
-    (area 42.709499 27.109499 68.0925 57.490501)
+    (area 42.044999 26.444999 282.27147 165.489573)
     (thickness 1.6002)
     (drawings 25)
@@
   (title_block
     (title "Multi Touch Bricklet")
-    (rev 1.0)
+    (date 2018-07-04)
+    (rev 2.0)
     (company "Tinkerforge GmbH")
     (comment 1 "Licensed under CERN OHL v.1.1")
-    (comment 2 "Copyright (©) 2013, B.Nordmeyer <bastian@tinkerforge.com>")
+    (comment 2 "Copyright (©) 2018, L.Lauer <lukas@tinkerforge.com>")
   )
   (layers
@@
   )
   (setup
-    (last_trace_width 0.25)
+    (last_trace_width 0.15)
     (user_trace_width 0.15)
     (user_trace_width 0.2)
@@
     (pad_to_mask_clearance 0)
     (aux_axis_origin 0 0)
-    (visible_elements FFFFFFBF)
+    (visible_elements FFFFEFBF)
     (pcbplotparams
       (layerselection 0x010fc_80000001)
@@
   (gr_arc (start 45.4 29.8) (end 42.9 29.8) (angle 90) (layer Edge.Cuts) (width 0.381))
   (gr_arc (start 45.4 54.8) (end 45.4 57.3) (angle 90) (layer Edge.Cuts) (width 0.381))
-  (gr_text "Copyright Tinkerforge GmbH 2013.\nThis documentation describes Open Hardware and is licensed under the\nCERN OHL v. 1.1.\nYou may redistribute and modify this documentation under the terms of the\nCERN OHL v.1.1. (http://ohwr.org/cernohl). This documentation is distributed\nWITHOUT ANY EXPRESS OR IMPLIED WARRANTY, INCLUDING OF\nMERCHANTABILITY, SATISFACTORY QUALITY AND FITNESS FOR A\nPARTICULAR PURPOSE. Please see the CERN OHL v.1.1 for applicable\nconditions" (at 258.32562 159.14878) (layer Cmts.User)
+  (gr_text "Copyright Tinkerforge GmbH 2018.\nThis documentation describes Open Hardware and is licensed under the\nCERN OHL v. 1.1.\nYou may redistribute and modify this documentation under the terms of the\nCERN OHL v.1.1. (http://ohwr.org/cernohl). This documentation is distributed\nWITHOUT ANY EXPRESS OR IMPLIED WARRANTY, INCLUDING OF\nMERCHANTABILITY, SATISFACTORY QUALITY AND FITNESS FOR A\nPARTICULAR PURPOSE. Please see the CERN OHL v.1.1 for applicable\nconditions" (at 258.32562 159.14878) (layer Cmts.User)
     (effects (font (size 0.8001 0.8001) (thickness 0.200025)))
   )

Commit message: Add 3d information
Other:
- rule trace_min: 0.15 -> 0
Changed lines of the file:
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@@
-(kicad_pcb (version 4) (host pcbnew 4.0.7+dfsg1-1ubuntu2)
+(kicad_pcb (version 4) (host pcbnew 4.0.2+dfsg1-stable)
   (general
     (links 69)
     (no_connects 0)
-    (area 42.044999 26.444999 282.27147 165.489573)
+    (area 42.709499 27.109499 68.0925 57.490501)
     (thickness 1.6002)
     (drawings 25)
@@
     (zone_clearance 0.24892)
     (zone_45_only no)
-    (trace_min 0.15)
+    (trace_min 0)
     (segment_width 0.381)
     (edge_width 0.381)
@@
     (pad 12 thru_hole circle (at 6.35 -1.27 90) (size 1.524 1.524) (drill 1.016) (layers *.Cu *.Mask F.SilkS)
       (net 23 "Net-(P4-Pad12)"))
-    (model Pin_Header/Pin_Header_Straight_2x06.wrl
-      (at (xyz 0.25 0.05 0))
+    (model Pin_Header/Pin_Header_Angled_2x6.wrl
+      (at (xyz 0 -0.05 0))
       (scale (xyz 1 1 1))
-      (rotate (xyz 0 0 90))
+      (rotate (xyz 0 0 0))
     )
   )

Commit message: Fix logos
Parts:
- moved VAL 8.96 mm to (55.4, 42.3)
- moved VAL 8.95 mm to (55.4, 49.8)
- moved G*** 8.93 mm to (55.4, 34.8)
Changed lines of the file:
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@@
   (title_block
     (title "Multi Touch Bricklet")
-    (date 2018-07-04)
+    (date 2018-07-06)
     (rev 2.0)
     (company "Tinkerforge GmbH")
@@
   )
   (module kicad-libraries:WEEE_7mm (layer Rückseite)
-    (at 46.44 42.58 180)
+    (at 55.4 42.3 180)
     (fp_text reference VAL (at 0 0 180) (layer B.SilkS) hide
       (effects (font (size 0.2 0.2) (thickness 0.05)) (justify mirror))
@@
   )
   (module kicad-libraries:CE_5mm (layer Rückseite)
-    (at 46.45 49.58 180)
+    (at 55.4 49.8 180)
     (fp_text reference VAL (at 0 0 180) (layer B.SilkS) hide
       (effects (font (size 0.2 0.2) (thickness 0.05)) (justify mirror))
@@
   )
   (module kicad-libraries:Logo_CoMCU (layer Rückseite)
-    (at 46.53 35.86 180)
+    (at 55.4 34.8 180)
     (fp_text reference G*** (at 0 0 180) (layer B.SilkS) hide
       (effects (font (thickness 0.3)) (justify mirror))
